File: hardware/motorpid.kicad_sch (KiCad schematic)
At the start: 112 parts, among them J1 BNC, J2 BNC, J3 BNC, J4 MOTOR + - shield, J5 POT 1 (+) 2 (wiper) 3 (-), J6 +15 / GND / -15, M1 fader motor, Q1 MJD44H11, Q2 MJD45H11, Q3 2N3904, Q4 2N3906, SW1 TARGET SOURCE, SW2 LOOP, SW3 D IN / OFF, SW4 I IN / OFF, SW5 D CAPACITOR, U1 LM321, U2 LM321, U3 LM321, U4 LM321, U5 LM321, U6 LM321, U7 LM321

Commit message: Simulate the loop from the exported netlist (ngspice, fader model); 22 nF D capacitor, 0.35 A fuse
Co-Authored-By: Claude Fable 5.1 <noreply@anthropic.com>
Claude-Session: https://claude.ai/code/session_017Q2PYKR2UewvTfQgKmRJsG
Parts:
- C5: value 10nF -> 22nF; LCSC C1710 -> C1729; MPN CL21B103KBANNNC -> CL21B223KBANNNC
- F1: value 0.5A -> 0.35A; LCSC C19078719 -> C18198328; MPN 1812L050/60GR -> 1812L035/30GR
Other:
- note added: "(T 0.6 s) use 100 nF and 1M. SW5 picks the capacitor,"
- note added: "0.35 A PTC opens a stall in seconds and resets itself."
- note added: "1: 22 nF, the slide pot"
- note added: "640k with the 22 nF; for the book's rotary motor-pot"
- note added: "MOTOR FUSE: 0.35 A resettable (not in the book)"
- note added: "SW3 puts D into the sum or shorts it out."
- note added: "Simulated as drawn (sim/pid_sim.py, the fader modelled from its data sheet): P only rings at 11 Hz when the gain"
- note added: "a stalled motor (0.6 A at full drive) trips it in 5-10 s; the"
- note added: "in 74 ms with 1 % overshoot. I removes the residual error at low P gain."
- note added: "nears 100; D equal to P there wants RC = 1 / 2 pi f = 14 ms (RV3 near 1414k with 22 nF), and then gain 100 settles"
- note added: "red lamp lights while it is tripped; it resets when the drive"
- note added: "stops. The loop runs the motor at 50-150 mA rms."
- note added: "the slide pot (T of 40-90 ms) that is 6-14 ms, 300k-"
- note added: "to 22 ms (22 nF), 100 ms (100 nF)"
- note removed: "0.5 A PTC opens a stall in seconds and resets itself."
- note removed: "1: 10 nF, the slide pot"
- note removed: "MOTOR FUSE: 0.5 A resettable (not in the book)"
- note removed: "With the slide pot the natural oscillation (P only, gain raised until it rings) is near 25 Hz; D equal to P"
- note removed: "a stalled motor (0.4-0.8 A) trips it in 10-30 s; the red"
- note removed: "lamp lights while it is tripped; it resets when the drive"
- note removed: "puts D into the sum or shorts it out."
- note removed: "stops. Running current is 0.1-0.3 A."
- note removed: "the 10 nF; for the book's rotary motor-pot (T 0.6 s)"
- note removed: "the slide pot (T about 40 ms) that is 6 ms, 600k with"
- note removed: "there wants RC = 1 / 2 pi f = 6 ms (RV3 at 640k with 10 nF). I removes the residual error at low P gain."
- note removed: "to 10 ms (10 nF), 100 ms (100 nF)"
- note removed: "use 100 nF and 1M. SW5 picks the capacitor, SW3"
Changed lines of the file:
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@@
 	)
 	(rectangle
-		(start 410.02 96.58)
-		(end 452.85 162.08)
+		(start 193.04 166.62)
+		(end 320.04 234.14)
 		(stroke
 			(width 0.15)
@@
 	)
 	(rectangle
-		(start 193.04 166.62)
-		(end 320.04 234.14)
+		(start 410.02 96.58)
+		(end 452.85 162.08)
 		(stroke
 			(width 0.15)
@@
 	)
 	(rectangle
-		(start 454.2 119.08)
-		(end 513.3 193.1)
+		(start 124.46 100.08)
+		(end 320.04 164.08)
 		(stroke
 			(width 0.15)
@@
 	)
 	(rectangle
-		(start 394.55 94.08)
-		(end 410.05 170.08)
+		(start 454.2 119.08)
+		(end 513.3 193.1)
 		(stroke
 			(width 0.15)
@@
 	)
 	(rectangle
-		(start 124.46 100.08)
-		(end 320.04 164.08)
+		(start 394.55 94.08)
+		(end 410.05 170.08)
 		(stroke
 			(width 0.15)
@@
 		)
 	)
+	(text "in 74 ms with 1 % overshoot.  I removes the residual error at low P gain."
+		(exclude_from_sim no)
+		(at 33.02 54.42 0)
+		(effects
+			(font
+				(size 1.5 1.5)
+			)
+			(justify left)
+		)
+	)
 	(text "Quiescent about 10 mA.  100 nF at every op-amp pin."
 		(exclude_from_sim no)
@@
 		)
 	)
+	(text "1: 22 nF, the slide pot"
+		(exclude_from_sim no)
+		(at 193.66 200.28 0)
+		(effects
+			(font
+				(size 1 1)
+			)
+			(justify left)
+		)
+	)
 	(text "PSEUDO OP-AMP: the book's home-made control amplifier, modest gain and no phase shift (Fig. 10L.6)"
 		(exclude_from_sim no)
@@
 		)
 	)
-	(text "use 100 nF and 1M.  SW5 picks the capacitor, SW3"
-		(exclude_from_sim no)
-		(at 238.76 353.035 0)
-		(effects
-			(font
-				(size 1.3 1.3)
-			)
-			(justify left)
-		)
-	)
 	(text "+15 V present"
 		(exclude_from_sim no)
@@
 		)
 	)
-	(text "stops.  Running current is 0.1-0.3 A."
-		(exclude_from_sim no)
-		(at 425.26 111.08 0)
-		(effects
-			(font
-				(size 1 1)
-			)
-			(justify left)
-		)
-	)
 	(text "CURRENT LIMIT and FUSE: not in the book.  1 ohm and a"
 		(exclude_from_sim no)
@@
 		)
 	)
+	(text "stops.  The loop runs the motor at 50-150 mA rms."
+		(exclude_from_sim no)
+		(at 425.26 111.08 0)
+		(effects
+			(font
+				(size 1 1)
+			)
+			(justify left)
+		)
+	)
 	(text "P = -ERROR"
 		(exclude_from_sim no)
@@
 		)
 	)
+	(text "to 22 ms (22 nF), 100 ms (100 nF)"
+		(exclude_from_sim no)
+		(at 231.14 219.28 0)
+		(effects
+			(font
+				(size 1.1 1.1)
+			)
+			(justify left)
+		)
+	)
 	(text "U1 takes TARGET - POSITION with four 100k.  U2 inverts"
 		(exclude_from_sim no)
@@
 		)
 	)
-	(text "puts D into the sum or shorts it out."
-		(exclude_from_sim no)
-		(at 238.76 355.57 0)
-		(effects
-			(font
-				(size 1.3 1.3)
-			)
-			(justify left)
-		)
-	)
 	(text "TARGET"
 		(exclude_from_sim no)
@@
 		)
 	)
-	(text "the other, 2 to the wiper; MOTOR + and - so that a"
+	(text "Simulated as drawn (sim/pid_sim.py, the fader modelled from its data sheet): P only rings at 11 Hz when the gain"
 		(exclude_from_sim no)
-		(at 457.2 347.965 0)
+		(at 33.02 48.22 0)
 		(effects
 			(font
-				(size 1.3 1.3)
+				(size 1.5 1.5)
 			)
 			(justify left)
 		)
 	)
-	(text "PID MOTOR CONTROL LOOP"
+	(text "the other, 2 to the wiper; MOTOR + and - so that a"
 		(exclude_from_sim no)
-		(at 33.02 20.32 0)
+		(at 457.2 347.965 0)
 		(effects
 			(font
-				(size 1.5 1.5)
+				(size 1.3 1.3)
 			)
 			(justify left)
 		)
 	)
-	(text "there wants RC = 1 / 2 pi f = 6 ms (RV3 at 640k with 10 nF).  I removes the residual error at low P gain."
+	(text "PID MOTOR CONTROL LOOP"
 		(exclude_from_sim no)
-		(at 33.02 51.32 0)
+		(at 33.02 20.32 0)
 		(effects
 			(font
@@
 		)
 	)
-	(text "the 10 nF; for the book's rotary motor-pot (T 0.6 s)"
-		(exclude_from_sim no)
-		(at 238.76 350.5 0)
-		(effects
-			(font
-				(size 1.3 1.3)
-			)
-			(justify left)
-		)
-	)
 	(text "Knob or jack, on the TARGET SOURCE switch.  The knob's"
 		(exclude_from_sim no)
@@
 		)
 	)
-	(text "to 10 ms (10 nF), 100 ms (100 nF)"
+	(text "SW1  TARGET SOURCE"
 		(exclude_from_sim no)
-		(at 231.14 219.28 0)
+		(at 84.44 121.58 0)
 		(effects
 			(font
@@
 		)
 	)
-	(text "lamp lights while it is tripped; it resets when the drive"
+	(text "(T 0.6 s) use 100 nF and 1M.  SW5 picks the capacitor,"
 		(exclude_from_sim no)
-		(at 425.26 109.08 0)
+		(at 238.76 353.035 0)
 		(effects
 			(font
-				(size 1 1)
+				(size 1.3 1.3)
 			)
 			(justify left)
 		)
 	)
-	(text "SW1  TARGET SOURCE"
+	(text "drives a second potentiometer to match it, and the controller is the book's home-made 'pseudo op-amp' of modest, adjustable"
 		(exclude_from_sim no)
-		(at 84.44 121.58 0)
+		(at 33.02 29.62 0)
 		(effects
 			(font
-				(size 1.1 1.1)
+				(size 1.5 1.5)
 			)
 			(justify left)
 		)
 	)
-	(text "drives a second potentiometer to match it, and the controller is the book's home-made 'pseudo op-amp' of modest, adjustable"
+	(text "640k with the 22 nF; for the book's rotary motor-pot"
 		(exclude_from_sim no)
-		(at 33.02 29.62 0)
+		(at 238.76 350.5 0)
 		(effects
 			(font
-				(size 1.5 1.5)
+				(size 1.3 1.3)
+			)
+			(justify left)
+		)
+	)
+	(text "the slide pot (T of 40-90 ms) that is 6-14 ms, 300k-"
+		(exclude_from_sim no)
+		(at 238.76 347.965 0)
+		(effects
+			(font
+				(size 1.3 1.3)
 			)
 			(justify left)
@@
 		)
 	)
-	(text "the slide pot (T about 40 ms) that is 6 ms, 600k with"
-		(exclude_from_sim no)
-		(at 238.76 347.965 0)
-		(effects
-			(font
-				(size 1.3 1.3)
-			)
-			(justify left)
-		)
-	)
 	(text "ERROR = TARGET - POSITION"
 		(exclude_from_sim no)
@@
 		)
 	)
-	(text "1: 10 nF, the slide pot"
+	(text "a stalled motor (0.6 A at full drive) trips it in 5-10 s; the"
 		(exclude_from_sim no)
-		(at 193.66 200.28 0)
+		(at 425.26 107.08 0)
 		(effects
 			(font
@@
 		)
 	)
-	(text "0.5 A PTC opens a stall in seconds and resets itself."
-		(exclude_from_sim no)
-		(at 345.44 370.78 0)
-		(effects
-			(font
-				(size 1.3 1.3)
-			)
-			(justify left)
-		)
-	)
 	(text "through 270 ohm and the 10k takes the feedback from the"
 		(exclude_from_sim no)
@@
 		)
 	)
+	(text "0.35 A PTC opens a stall in seconds and resets itself."
+		(exclude_from_sim no)
+		(at 345.44 370.78 0)
+		(effects
+			(font
+				(size 1.3 1.3)
+			)
+			(justify left)
+		)
+	)
 	(text "At P gain 1.5 the loop is stable and slow; near 20 it"
 		(exclude_from_sim no)
@@
 		)
 	)
+	(text "nears 100; D equal to P there wants RC = 1 / 2 pi f = 14 ms (RV3 near 1414k with 22 nF), and then gain 100 settles"
+		(exclude_from_sim no)
+		(at 33.02 51.32 0)
+		(effects
+			(font
+				(size 1.5 1.5)
+			)
+			(justify left)
+		)
+	)
 	(text "follower"
 		(exclude_from_sim no)
@@
 		)
 	)
+	(text "red lamp lights while it is tripped; it resets when the drive"
+		(exclude_from_sim no)
+		(at 425.26 109.08 0)
+		(effects
+			(font
+				(size 1 1)
+			)
+			(justify left)
+		)
+	)
+	(text "MOTOR FUSE: 0.35 A resettable (not in the book)"
+		(exclude_from_sim no)
+		(at 425.26 105.08 0)
+		(effects
+			(font
+				(size 1.2 1.2)
+			)
+			(justify left)
+		)
+	)
 	(text "POSITION OUT"
 		(exclude_from_sim no)
@@
 		)
 	)
+	(text "SW3 puts D into the sum or shorts it out."
+		(exclude_from_sim no)
+		(at 238.76 355.57 0)
+		(effects
+			(font
+				(size 1.3 1.3)
+			)
+			(justify left)
+		)
+	)
 	(text "Op-amps are drawn + on top: that is how the SOT-23-5 sits."
 		(exclude_from_sim no)
@@
 		)
 	)
-	(text "a stalled motor (0.4-0.8 A) trips it in 10-30 s; the red"
-		(exclude_from_sim no)
-		(at 425.26 107.08 0)
-		(effects
-			(font
-				(size 1 1)
-			)
-			(justify left)
-		)
-	)
 	(text "I = -(1/RC) integral of ERROR dt"
 		(exclude_from_sim no)
@@
 		)
 	)
-	(text "MOTOR FUSE: 0.5 A resettable (not in the book)"
-		(exclude_from_sim no)
-		(at 425.26 105.08 0)
-		(effects
-			(font
-				(size 1.2 1.2)
-			)
-			(justify left)
-		)
-	)
 	(text "drives the residual error to zero; too much I rings."
 		(exclude_from_sim no)
@@
 		)
 	)
-	(text "With the slide pot the natural oscillation (P only, gain raised until it rings) is near 25 Hz; D equal to P"
-		(exclude_from_sim no)
-		(at 33.02 48.22 0)
-		(effects
-			(font
-				(size 1.5 1.5)
-			)
-			(justify left)
-		)
-	)
 	(text "P GAIN: (10k + RV2) / 10k"
 		(exclude_from_sim no)
@@
 			)
 		)
-		(property "Value" "0.5A"
+		(property "Value" "0.35A"
 			(at 436.88 137.08 90)
 			(show_name no)
@@
 			)
 		)
-		(property "LCSC" "C19078719"
+		(property "LCSC" "C18198328"
 			(at 436.88 132.08 90)
 			(hide yes)
@@
 			)
 		)
-		(property "MPN" "1812L050/60GR"
+		(property "MPN" "1812L035/30GR"
 			(at 436.88 132.08 90)
 			(hide yes)
@@
 			)
 		)
-		(property "Value" "10nF"
+		(property "Value" "22nF"
 			(at 190.5 202.94 90)
 			(show_name no)
@@
 			)
 		)
-		(property "LCSC" "C1710"
+		(property "LCSC" "C1729"
 			(at 190.5 205.74 90)
 			(hide yes)
@@
 			)
 		)
-		(property "MPN" "CL21B103KBANNNC"
+		(property "MPN" "CL21B223KBANNNC"
 			(at 190.5 205.74 90)
 			(hide yes)

Commit message: Move TARGET IN BNC off the knob's wire column (its shield grounded the knob's bottom end); add shorted-part and knob-end netlist checks
Co-Authored-By: Claude Fable 5.1 <noreply@anthropic.com>
Claude-Session: https://claude.ai/code/session_017Q2PYKR2UewvTfQgKmRJsG
Connections:
- net GND: no longer C2.2, R2.1, RV1.3
- new net: C2.2, R2.1, RV1.3
Other:
- note added: "(±0.5 V at 0.2 Hz) replaces the knob"
- note added: "in 92 ms with 1 % overshoot. I removes the residual error at low P gain."
- note added: "nears 100; D equal to P there wants RC = 1 / 2 pi f = 14 ms (RV3 near 643k with 22 nF), and then gain 100 settles"
- note added: "±12 V max; a slow square wave"
- note removed: "in 74 ms with 1 % overshoot. I removes the residual error at low P gain."
- note removed: "nears 100; D equal to P there wants RC = 1 / 2 pi f = 14 ms (RV3 near 1414k with 22 nF), and then gain 100 settles"
- note removed: "±12 V max; a slow square wave (±0.5 V at 0.2 Hz) replaces the knob"
- moved on the sheet: J1
Changed lines of the file:
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@@
 	)
 	(rectangle
-		(start 193.04 166.62)
-		(end 320.04 234.14)
+		(start 193.04 237.74)
+		(end 320.04 305.26)
 		(stroke
 			(width 0.15)
@@
 	)
 	(rectangle
-		(start 193.04 237.74)
-		(end 320.04 305.26)
+		(start 394.55 94.08)
+		(end 410.05 170.08)
 		(stroke
 			(width 0.15)
@@
 	)
 	(rectangle
-		(start 410.02 96.58)
-		(end 452.85 162.08)
+		(start 193.04 166.62)
+		(end 320.04 234.14)
 		(stroke
 			(width 0.15)
@@
 	)
 	(rectangle
-		(start 394.55 94.08)
-		(end 410.05 170.08)
+		(start 410.02 96.58)
+		(end 452.85 162.08)
 		(stroke
 			(width 0.15)
@@
 		)
 	)
-	(text "in 74 ms with 1 % overshoot.  I removes the residual error at low P gain."
-		(exclude_from_sim no)
-		(at 33.02 54.42 0)
-		(effects
-			(font
-				(size 1.5 1.5)
-			)
-			(justify left)
-		)
-	)
 	(text "Quiescent about 10 mA.  100 nF at every op-amp pin."
 		(exclude_from_sim no)
@@
 		)
 	)
+	(text "(±0.5 V at 0.2 Hz) replaces the knob"
+		(exclude_from_sim no)
+		(at 33.02 147.066 0)
+		(effects
+			(font
+				(size 1.1 1.1)
+			)
+			(justify left)
+		)
+	)
 	(text "= 1 to 101"
 		(exclude_from_sim no)
@@
 		)
 	)
+	(text "TARGET IN"
+		(exclude_from_sim no)
+		(at 33.02 139.7 0)
+		(effects
+			(font
+				(size 2.2 2.2)
+			)
+			(justify left)
+		)
+	)
 	(text "D = -RV3 C dERROR/dt, rolled off above 500 Hz by the"
 		(exclude_from_sim no)
@@
 		)
 	)
-	(text "nears 100; D equal to P there wants RC = 1 / 2 pi f = 14 ms (RV3 near 1414k with 22 nF), and then gain 100 settles"
+	(text "nears 100; D equal to P there wants RC = 1 / 2 pi f = 14 ms (RV3 near 643k with 22 nF), and then gain 100 settles"
 		(exclude_from_sim no)
 		(at 33.02 51.32 0)
@@
 		)
 	)
+	(text "±12 V max; a slow square wave"
+		(exclude_from_sim no)
+		(at 33.02 144.018 0)
+		(effects
+			(font
+				(size 1.1 1.1)
+			)
+			(justify left)
+		)
+	)
 	(text "A ±0.5 V square wave at 0.2 Hz from a generator on the"
 		(exclude_from_sim no)
@@
 		)
 	)
+	(text "in 92 ms with 1 % overshoot.  I removes the residual error at low P gain."
+		(exclude_from_sim no)
+		(at 33.02 54.42 0)
+		(effects
+			(font
+				(size 1.5 1.5)
+			)
+			(justify left)
+		)
+	)
 	(text "stays inside the rails"
 		(exclude_from_sim no)
@@
 		)
 	)
-	(text "TARGET IN"
-		(exclude_from_sim no)
-		(at 33.02 143.51 0)
-		(effects
-			(font
-				(size 2.2 2.2)
-			)
-			(justify left)
-		)
-	)
 	(text "-90 degrees would make -180 at a few hertz.  The pseudo op-amp has gain 1 to 101 and no phase shift of its own."
 		(exclude_from_sim no)
@@
 		)
 	)
-	(text "±12 V max; a slow square wave (±0.5 V at 0.2 Hz) replaces the knob"
-		(exclude_from_sim no)
-		(at 33.02 147.828 0)
-		(effects
-			(font
-				(size 1.1 1.1)
-			)
-			(justify left)
-		)
-	)
 	(text "barely limited."
 		(exclude_from_sim no)
@@
 	)
 	(junction
-		(at 55.88 160.02)
-		(diameter 0)
-		(color 0 0 0 0)
-	)
-	(junction
 		(at 172.72 157.48)
 		(diameter 0)
@@
 	)
 	(junction
-		(at 55.88 167.64)
-		(diameter 0)
-		(color 0 0 0 0)
-	)
-	(junction
 		(at 414.02 325.12)
 		(diameter 0)
@@
 	(wire
 		(pts
-			(xy 60.96 154.94) (xy 83.82 154.94)
-		)
-		(stroke
-			(width 0)
-			(type default)
-		)
-	)
-	(wire
-		(pts
 			(xy 205.74 134.62) (xy 205.74 142.24)
 		)
@@
 	(wire
 		(pts
+			(xy 48.26 154.94) (xy 83.82 154.94)
+		)
+		(stroke
+			(width 0)
+			(type default)
+		)
+	)
+	(wire
+		(pts
 			(xy 266.7 302.26) (xy 220.98 302.26)
 		)
@@
 	(wire
 		(pts
-			(xy 55.88 160.02) (xy 55.88 167.64)
-		)
-		(stroke
-			(width 0)
-			(type default)
-		)
-	)
-	(wire
-		(pts
 			(xy 220.98 231.14) (xy 220.98 208.28)
 		)
@@
 	(wire
 		(pts
+			(xy 43.18 160.02) (xy 43.18 167.64)
+		)
+		(stroke
+			(width 0)
+			(type default)
+		)
+	)
+	(wire
+		(pts
 			(xy 474.98 162.56) (xy 474.98 154.94)
 		)
@@
 		)
 	)
-	(label "TARGET IN"
-		(at 66.04 154.94 0)
-		(effects
-			(font
-				(size 1.3 1.3)
-			)
-			(justify left)
-		)
-	)
 	(label "I"
 		(at 250.42 269.24 0)
@@
 		)
 	)
+	(label "TARGET IN"
+		(at 53.34 154.94 0)
+		(effects
+			(font
+				(size 1.3 1.3)
+			)
+			(justify left)
+		)
+	)
 	(label "BASES"
 		(at 375.92 132.08 0)
@@
 	(symbol
 		(lib_id "power:GND")
-		(at 55.88 167.64 0)
+		(at 43.18 167.64 0)
 		(unit 1)
 		(body_style 1)
@@
 		(dnp no)
 		(property "Reference" "#PWR0003"
-			(at 55.88 160.02 0)
+			(at 43.18 160.02 0)
 			(hide yes)
 			(show_name no)
@@
 		)
 		(property "Value" "GND"
-			(at 55.88 175.26 0)
+			(at 43.18 175.26 0)
 			(hide yes)
 			(show_name no)
@@
 		)
 		(property "Footprint" ""
-			(at 55.88 167.64 0)
+			(at 43.18 167.64 0)
 			(hide yes)
 			(show_name no)
@@
 		)
 		(property "Datasheet" ""
-			(at 55.88 167.64 0)
+			(at 43.18 167.64 0)
 			(hide yes)
 			(show_name no)
@@
 		)
 		(property "Description" ""
-			(at 55.88 167.64 0)
+			(at 43.18 167.64 0)
 			(hide yes)
 			(show_name no)
@@
 	(symbol
 		(lib_id "Connector:Conn_Coaxial")
-		(at 55.88 154.94 0)
+		(at 43.18 154.94 0)
 		(mirror y)
 		(unit 1)
@@
 		(dnp no)
 		(property "Reference" "J1"
-			(at 51.88 156.54 0)
+			(at 39.18 156.54 0)
 			(show_name no)
 			(do_not_autoplace no)
@@
 		)
 		(property "Value" "BNC"
-			(at 51.88 158.34 0)
+			(at 39.18 158.34 0)
 			(show_name no)
 			(do_not_autoplace no)
@@
 		)
 		(property "Footprint" "motorpid:BNC_KYWE_RightAngle"
-			(at 55.88 154.94 0)
+			(at 43.18 154.94 0)
 			(hide yes)
 			(show_name no)
@@
 		)
 		(property "Datasheet" ""
-			(at 55.88 154.94 0)
+			(at 43.18 154.94 0)
 			(hide yes)
 			(show_name no)
@@
 		)
 		(property "Description" ""
-			(at 55.88 154.94 0)
+			(at 43.18 154.94 0)
 			(hide yes)
 			(show_name no)
@@
 		)
 		(property "LCSC" "C41416668"
-			(at 55.88 154.94 0)
+			(at 43.18 154.94 0)
 			(hide yes)
 			(show_name no)
@@
 		)
 		(property "MPN" "BNC-KYWE-295-W4-N"
-			(at 55.88 154.94 0)
+			(at 43.18 154.94 0)
 			(hide yes)
 			(show_name no)

Commit message: Drop the output current limiter (the PTC is the protection; the 1 ohm emitter resistors stay as current sense); knob pin 3 on the + end so clockwise is positive; make.py for this project
Co-Authored-By: Claude Fable 5.1 <noreply@anthropic.com>
Claude-Session: https://claude.ai/code/session_017Q2PYKR2UewvTfQgKmRJsG
Parts:
- removed D5, D6: 1N4148W, Diode_SMD:D_SOD-123, symbol Device:D
- removed Q3: 2N3904, Package_TO_SOT_SMD:SOT-23, symbol Transistor_BJT:MMBT3904
- removed Q4: 2N3906, Package_TO_SOT_SMD:SOT-23, symbol Transistor_BJT:MMBT3906
Connections:
- net at C2.2, R2.1: now also RV1.1; no longer RV1.3
- net at C1.1, R1.2: now also RV1.3; no longer RV1.1
Other:
- note added: "(0.6 A) in seconds and a short in well under one, then"
- note added: "1 V per ampere of motor current, for a scope."
- note added: "FUSE: not in the book. The 0.35 A PTC opens a stall"
- note added: "R21, R22: 1 ohm, not in the book. Across either one,"
- note added: "knob, centre detent = 0 V, clockwise = +"
- note added: "resets itself when it cools. 1 ohm per emitter reads"
- note added: "the motor current: 1 V per A across R21 or R22."
- note removed: "0.35 A PTC opens a stall in seconds and resets itself."
- note removed: "0.65 V across 1 ohm turns Q3 (Q4)"
- note removed: "CURRENT LIMIT and FUSE: not in the book. 1 ohm and a"
- note removed: "OUTPUT CURRENT LIMIT"
- note removed: "barely limited."
- note removed: "for seconds; a stall (0.4-0.8 A) is"
- note removed: "knob, centre detent = 0 V"
- note removed: "not in the book: a safety net."
- note removed: "on and it steals the drive: 0.65 A,"
- note removed: "small transistor per half hold a short to 0.65 A; the"
- note removed: "so a shorted MOTOR terminal lives"
