File: hardware/motorpid.kicad_sch (KiCad schematic)
At the start: 111 parts, among them J1 BNC, J2 BNC, J3 BNC, J4 MOTOR + - shield, J5 POT 1 (+) 2 (wiper) 3 (-), J6 +15 / GND / -15, M1 fader motor, Q1 MJD44H11, Q2 MJD45H11, SW1 TARGET SOURCE, SW2 LOOP, SW3 D IN / OFF, SW4 I IN / OFF, SW5 D CAPACITOR, U1 LM321, U2 LM321, U3 LM321, U4 LM321, U5 LM321, U6 LM321, U7 LM321

Commit message: Push-pull on D2PAKs and 2 oz copper (Jason's choice): MJB44H11/MJB45H11 in pours that are their heatsink, 120/122 C junctions in the worst stall, checked on the board as built
- parts: MJB44H11T4G C233689 / MJB45H11T4G C154570, TO-263-2; JLCPCB draws
  them turned 180 (CPL +180, datum 2.45 mm toward the leads, predicted)
- layout: Q1/Q2 symbols drawn round the leads with the tab capping the
  circle; pours fill the MOTOR DRIVER box round each tab (836 / 670 mm2);
  R21/R22 in two columns; D3/D4 with their rail ends in the pours; snubber
  under DRIVE; BASES crosses Q2's emitter wire on the back (one hop: the
  mirrored PNP makes the crossing topological)
- back runs moved off the plane under the pours: lower stages' +15 V from
  the rail, Q2's -15 V up the board edge, U6 V- and the track's -15 V from
  Q2's pour
- 2 oz: clearance and min track 0.21 mm, board stackup 0.07 mm copper,
  order form says 2 oz, bare-board cost x1.5
- sim/thermal.py --board: the model on the filled pours and the plane with
  its cuts; make.py fails above 125 C at the junction; sim/thermal.json
- pid_sim refuses a transistor it has no model for (a stale netlist
  silently simulated the wrong part once)
- docs: decision recorded, 5 new build-checked claims, HOT on both pours,
  warnings softened from "seconds" to "the copper is hot"

ERC 0, 249 checks, DRC 0, fab checks, 30/30 claims, BUILD OK.

Co-Authored-By: Claude Opus 5.5 <noreply@anthropic.com>
Claude-Session: https://claude.ai/code/session_017Q2PYKR2UewvTfQgKmRJsG
Parts:
- Q1: value MJD44H11 -> MJB44H11; footprint Package_TO_SOT_SMD:TO-252-2 -> Package_TO_SOT_SMD:TO-263-2; LCSC C38780 -> C233689; MPN MJD44H11T4G -> MJB44H11T4G
- Q2: value MJD45H11 -> MJB45H11; footprint Package_TO_SOT_SMD:TO-252-2 -> Package_TO_SOT_SMD:TO-263-2; LCSC C47515 -> C154570; MPN MJD45H11T4G -> MJB45H11T4G
Other:
- note added: "2 oz copper pours. R21, R22 read the motor current, 1 V/A."
- note added: "and stalls there, heating the driver: TARGET back to 0."
- note added: "one transistor takes up to 3.7 W, so they are D2PAKs on"
- note added: "own LM321 (the single LM358), the book's MJE3055/2955 as D2PAK MJB44H11/45H11, and its resistor substitution boxes as trimmers."
- note removed: "a transistor takes up to 3.7 W. 1 ohm per emitter reads"
- note removed: "and stalls there: bring TARGET back to 0 within seconds."
- note removed: "own LM321 (the single LM358), the book's MJE3055/2955 as DPAK MJD44H11/45H11, and its resistor substitution boxes as trimmers."
- note removed: "the motor current: 1 V per A across R21 or R22."
Changed lines of the file:
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@@
 		(rev "A")
 		(company "Circuit: Hayes & Horowitz, Learning the Art of Electronics (2016), Lab 10L  |  Board: Jason Gallicchio and Claude")
-		(comment 1 "LM321 (the single LM358) in SOT-23-5, one per triangle; MJD44H11 / MJD45H11 push-pull")
+		(comment 1 "LM321 (the single LM358) in SOT-23-5, one per triangle; MJB44H11 / MJB45H11 (D2PAK) push-pull")
 		(comment 2 "P from 1 to 101, D up to 10 ms (slide pot) or 100 ms (rotary), I up to 10 s")
 		(comment 3 "Open source, CERN-OHL-P-2.0 -- github.com/gallicchio/motor-pid")
 	)
 	(rectangle
-		(start 193.04 237.74)
-		(end 320.04 305.26)
+		(start 410.02 96.58)
+		(end 452.85 162.08)
 		(stroke
 			(width 0.15)
@@
 	)
 	(rectangle
-		(start 193.04 166.62)
-		(end 320.04 234.14)
+		(start 124.46 100.08)
+		(end 320.04 164.08)
 		(stroke
 			(width 0.15)
@@
 	)
 	(rectangle
-		(start 124.46 100.08)
-		(end 320.04 164.08)
+		(start 454.2 119.08)
+		(end 513.3 193.1)
 		(stroke
 			(width 0.15)
@@
 	)
 	(rectangle
-		(start 454.2 119.08)
-		(end 513.3 193.1)
+		(start 193.04 166.62)
+		(end 320.04 234.14)
 		(stroke
 			(width 0.15)
@@
 	)
 	(rectangle
-		(start 410.02 96.58)
-		(end 452.85 162.08)
+		(start 193.04 237.74)
+		(end 320.04 305.26)
 		(stroke
 			(width 0.15)
@@
 		)
 	)
-	(text "and stalls there: bring TARGET back to 0 within seconds."
-		(exclude_from_sim no)
-		(at 33.02 373.315 0)
-		(effects
-			(font
-				(size 1.3 1.3)
-			)
-			(justify left)
-		)
-	)
 	(text "P = -ERROR"
 		(exclude_from_sim no)
@@
 		)
 	)
-	(text "the motor current: 1 V per A across R21 or R22."
-		(exclude_from_sim no)
-		(at 345.44 375.85 0)
-		(effects
-			(font
-				(size 1.3 1.3)
-			)
-			(justify left)
-		)
-	)
 	(text "THE PLANT: motor and pot  (Fig. 10L.1)"
 		(exclude_from_sim no)
@@
 		)
 	)
+	(text "one transistor takes up to 3.7 W, so they are D2PAKs on"
+		(exclude_from_sim no)
+		(at 345.44 373.315 0)
+		(effects
+			(font
+				(size 1.3 1.3)
+			)
+			(justify left)
+		)
+	)
 	(text "summing amplifier, gain -Rgain/10k"
 		(exclude_from_sim no)
@@
 		)
 	)
-	(text "own LM321 (the single LM358), the book's MJE3055/2955 as DPAK MJD44H11/45H11, and its resistor substitution boxes as trimmers."
+	(text "own LM321 (the single LM358), the book's MJE3055/2955 as D2PAK MJB44H11/45H11, and its resistor substitution boxes as trimmers."
 		(exclude_from_sim no)
 		(at 33.02 35.82 0)
@@
 		)
 	)
+	(text "and stalls there, heating the driver: TARGET back to 0."
+		(exclude_from_sim no)
+		(at 33.02 373.315 0)
+		(effects
+			(font
+				(size 1.3 1.3)
+			)
+			(justify left)
+		)
+	)
+	(text "2 oz copper pours.  R21, R22 read the motor current, 1 V/A."
+		(exclude_from_sim no)
+		(at 345.44 375.85 0)
+		(effects
+			(font
+				(size 1.3 1.3)
+			)
+			(justify left)
+		)
+	)
 	(text "nears 100; D equal to P there wants RC = 1 / 2 pi f = 5 ms (RV3 near 234k with 22 nF), and then gain 100 settles"
 		(exclude_from_sim no)
@@
 		)
 	)
-	(text "a transistor takes up to 3.7 W.  1 ohm per emitter reads"
-		(exclude_from_sim no)
-		(at 345.44 373.315 0)
-		(effects
-			(font
-				(size 1.3 1.3)
-			)
-			(justify left)
-		)
-	)
 	(text "R21, R22: 1 ohm, not in the book.  Across either one,"
 		(exclude_from_sim no)
@@
 			)
 		)
-		(property "Value" "MJD45H11"
+		(property "Value" "MJB45H11"
 			(at 394.22 157.94 0)
 			(show_name no)
@@
 			)
 		)
-		(property "Footprint" "Package_TO_SOT_SMD:TO-252-2"
+		(property "Footprint" "Package_TO_SOT_SMD:TO-263-2"
 			(at 388.62 154.94 0)
 			(hide yes)
@@
 			)
 		)
-		(property "LCSC" "C47515"
+		(property "LCSC" "C154570"
 			(at 388.62 154.94 0)
 			(hide yes)
@@
 			)
 		)
-		(property "MPN" "MJD45H11T4G"
+		(property "MPN" "MJB45H11T4G"
 			(at 388.62 154.94 0)
 			(hide yes)
@@
 			)
 		)
-		(property "Value" "MJD44H11"
+		(property "Value" "MJB44H11"
 			(at 394.22 108.62 0)
 			(show_name no)
@@
 			)
 		)
-		(property "Footprint" "Package_TO_SOT_SMD:TO-252-2"
+		(property "Footprint" "Package_TO_SOT_SMD:TO-263-2"
 			(at 388.62 109.22 0)
 			(hide yes)
@@
 			)
 		)
-		(property "LCSC" "C38780"
+		(property "LCSC" "C233689"
 			(at 388.62 109.22 0)
 			(hide yes)
@@
 			)
 		)
-		(property "MPN" "MJD44H11T4G"
+		(property "MPN" "MJB44H11T4G"
 			(at 388.62 109.22 0)
 			(hide yes)

Commit message: Review round 1 applied (Jason): the patch, the fuse between the push-pull and DRIVE, the integrator's capacitor a 1 uF polypropylene film
- patch_round1.diff as it stood: switch-end numbers, three vias each end of Q2's -15 V run,
  TARGET IN at +/-3 V, standoffs, handbook table and gains recipe, R4's run off the URL,
  sheet notes; its "DRIVE ahead of the fuse" warnings rewritten for the moved fuse
- F1 right after R21/R22: the feedback, the DRIVE loop, DRIVE OUT and the motor terminal
  behind it; clamps and snubber stay at the transistors; MOTOR merged into DRIVE (17 loops);
  check_circuit asserts what is ahead of the fuse and that no loop or connector is
- C8: Panasonic ECWF2W105JA 1 uF PP film (C242107), generated footprint and model; RC 1 ms
  to 1 s across the 1M trimmer; the LM321's bias current through 1M (45 mV) in a check
- sim: motor on DRIVE, Q1's power from its own pins (3.4 W; the old 3.7 included R21),
  I runs at 1M and 50k; thermal check keeps 3.7 W as a bound, 120/122 C
- fab notes: D4's cathode and C12's stripe were drawn the wrong way; the 1R's BOM note
- the review brief describes the patched board; reviews README and the report's addendum
- ERC 0, 252 checks, DRC 0, fab checks, 30/30 claims

Co-Authored-By: Claude Opus 5.5 <noreply@anthropic.com>
Claude-Session: https://claude.ai/code/session_017Q2PYKR2UewvTfQgKmRJsG
Parts:
- removed TP14: U7 OUT, motorpid:TestPoint_Loop_RH-5019, symbol Connector:TestPoint
- C8: value 10uF -> 1uF; footprint Capacitor_SMD:C_0805_2012Metric -> motorpid:C_Film_Panasonic_ECWF_L18.1mm_W9.3mm_P15.00mm; LCSC C15850 -> C242107; MPN CL21A106KAYNNNE -> ECWF2W105JA
- TP11: value MOTOR -> BASES
- TP12: value BASES -> U6 OUT
- TP13: value U6 OUT -> U7 OUT
Connections:
- net BASES: now also TP11.1; no longer TP12.1
- net DRIVE: now also F1.2, J4.1 (Pin_1), LED3.2 (A), LED4.1 (K), M1.1 (+); no longer D3.2 (A), D4.1 (K), F1.1, R20.1, R21.2, R22.1, R23.1
- net at R25.1, U7.3 (-), U7.4: now also TP13.1
- net at C9.2, R19.1, U6.4: now also TP12.1; no longer TP13.1
- removed net MOTOR: F1.2, J4.1 (Pin_1), LED3.2 (A), LED4.1 (K), M1.1 (+), TP11.1
- new net: D3.2 (A), D4.1 (K), F1.1, R20.1, R21.2, R22.1, R23.1
Other:
- note added: "(0.6 A) trips it in 5-10 s, a short in"
- note added: "1 ms to 1 s"
- note added: "231k with the 22 nF; for the book's rotary motor-pot"
- note added: "D = -RV3 C dERROR/dt, rolled off by the 470 pF (1.5 kHz"
- note added: "D3, D4 clamp the motor's inductive kick"
- note added: "FUSE 0.35 A, resettable"
- note added: "FUSE: not in the book. Between the push-pull and DRIVE:"
- note added: "I = -(1/RC) integral ERROR dt, RC = (1k + RV4) x 1 uF,"
- note added: "I GAIN: RC = (1k + RV4) x 1 uF"
- note added: "a polypropylene film: its value holds at any voltage."
- note added: "about 1 s; the red lamp lights while it"
- note added: "at a few volts it holds: one transistor takes up to 3.4 W,"
- note added: "at the rule). Set RV3 C to 1/6 of the natural period: for"
- note added: "behind it. The 0.35 A PTC opens a full-drive stall (0.6 A)"
- note added: "differentiator; 470 pF rolls it off, 1.5 kHz at the rule"
- note added: "film"
- note added: "in seconds and a short in about one, then resets. A stall"
- note added: "is tripped. It resets when the drive stops."
- note added: "nears 100; D equal to P there wants RC = 1 / 2 pi f = 5 ms (RV3 near 231k with 22 nF), and then gain 100 settles"
- note added: "not in the book. A stall at full drive"
- note added: "per ampere: two probes, A - B (never a ground clip there)."
- note added: "so they are D2PAKs on 2 oz pours. Across R21 or R22, 1 V"
- note added: "the brush hash. ±13 V unloaded, ±9 V into a stall; 10 V motor,"
- note added: "the feedback, the DRIVE loop, DRIVE OUT and the motor are"
- note added: "the motor's voltage"
- note added: "through 1k: ±13 V"
- note added: "to the rails, at the transistors"
- note added: "±13 V, 0.35 A fuse"
- note removed: "1 V per ampere of motor current, for a scope."
- note removed: "10 ms to 10 s"
- note removed: "2 oz copper pours. R21, R22 read the motor current, 1 V/A."
- note removed: "234k with the 22 nF; for the book's rotary motor-pot"
- note removed: "470 pF. Set RV3 C to 1/6 of the natural period: for"
- note removed: "D = -RV3 C dERROR/dt, rolled off above 500 Hz by the"
- note removed: "D3, D4: clamps, so the motor's inductive kick"
- note removed: "FUSE: not in the book. The 0.35 A PTC opens a full-drive"
- note removed: "I = -(1/RC) integral ERROR dt, RC = (1k + RV4) x 10 uF."
- note removed: "I GAIN: RC = (1k + RV4) x 10 uF"
- note removed: "MOTOR FUSE: 0.35 A resettable (not in the book)"
- note removed: "R21, R22: 1 ohm, not in the book. Across either one,"
- note removed: "a stalled motor (0.6 A at full drive) trips it in 5-10 s; the"
- note removed: "differentiator; 470 pF rolls it off above 500 Hz"
- note removed: "nears 100; D equal to P there wants RC = 1 / 2 pi f = 5 ms (RV3 near 234k with 22 nF), and then gain 100 settles"
- note removed: "one transistor takes up to 3.7 W, so they are D2PAKs on"
- note removed: "red lamp lights while it is tripped; it resets when the drive"
- note removed: "stall (0.6 A) in seconds and a short in well under one,"
- note removed: "stays inside the rails"
- note removed: "stops. The loop runs the motor at 50-150 mA rms."
- note removed: "the brush hash. Output ±13 V; the motor is rated 10 V,"
- note removed: "the motor's voltage through 1k: ±13 V"
- note removed: "then resets itself. A stall at a few volts it holds, and"
- note removed: "±13 V, 0.65 A max"
- moved on the sheet: C10, D3, D4, F1, J3, LED3, LED4, R20, R23, R24

Commit message: Review round 1 closed: Gemini-4-Argon's and KimiK3's findings applied (RV1's JLCPCB rotation, the fuse's stall story and its 60 V grade, rail clamps D5/D6, the LM321's real swing, step metrics that name the dead band, silk dots and boxes, kienv and the sim's netlist, a deterministic sheet)
- RV1 (C351173): +270 and (3.5, -2.5); JLCPCB's drawing overlaid by the new CPL lands on our pins
- F1: LUTE 1812L035/60GR (C18198330), same hold/trip/R; every document now says a short opens it
  in about a second and a full-drive stall (0.61 A, between hold and trip) may take minutes or never
- D5, D6 (SS34) clamp each rail to ground: one rail left open cannot reverse-bias its electrolytic
- sim: LM321 output 2 V from each rail (D rule 239k, stall 0.61 A, step drive 11.7 V); step metrics
  report peak, swing back and rest separately; the sim stage exports its own netlist
- silk: dot where the dashed POSITION branches and at the track's end capacitors; C3/C4 inside
  their box; the -15 V flag clear of the title; D2PAK emitter copper at full width
- docs: the book's real "not 411", knob direction settled, scope grounds on GND loops only,
  x10 probes, the gains recipe's switches and signs, the rail-sag rest offset with the jack
- build: KiCad 9 on PATH no longer wins; rectangles' UUIDs hashed (byte-identical sheet);
  check messages from the sim; stock from the BOM; dead limiter parts removed
- the two reviews committed (the Fable-labelled one renamed KimiK3, Jason to confirm the
  model; datasheet excerpts kept out of git); the reviews README and the brief updated
- ERC 0, 258 checks, DRC 0, thermal 120/122 C, fab checks, 31/31 claims

Co-Authored-By: Claude Opus 5.5 <noreply@anthropic.com>
Claude-Session: https://claude.ai/code/session_017Q2PYKR2UewvTfQgKmRJsG
Parts:
- added D5, D6: SS34, Diode_SMD:D_SMA, symbol Device:D_Schottky
- F1: LCSC C18198328 -> C18198330; MPN 1812L035/30GR -> 1812L035/60GR
Connections:
- net +15V: now also D5.1 (K)
- net -15V: now also D6.2 (A)
- net GND: now also D5.2 (A), D6.1 (K)
Other:
- note added: "(±3 V at 0.2 Hz) replaces the knob"
- note added: "239k with the 22 nF; for the book's rotary motor-pot"
- note added: "D5, D6: clamps, if one rail is left open"
- note added: "POWER: ±15 V, 1 A. Series Schottkys block a reversed"
- note added: "Red lamps while it is open."
- note added: "Simulated as drawn (sim/pid_sim.py, the fader modelled from bench measurements): P only rings at 30 Hz when the gain"
- note added: "a D2PAK on a 2 oz pour. Across R21 or R22, 1 V per ampere:"
- note added: "about a second; a full-drive stall (0.6 A) is between its"
- note added: "behind it. The 0.35 A PTC opens a short of DRIVE (2 A) in"
- note added: "hold and trip and may take minutes; a stall at a few volts"
- note added: "in 29 ms with 3 % overshoot. I removes the residual error at low P gain."
- note added: "in about a second; a full-drive"
- note added: "may never open it: one transistor then carries up to 3.4 W,"
- note added: "nears 100; D equal to P there wants RC = 1 / 2 pi f = 5 ms (RV3 near 239k with 22 nF), and then gain 100 settles"
- note added: "not in the book. A short opens it"
- note added: "op-amp pin. Quiescent about 4 mA."
- note added: "stall (0.6 A) can take minutes."
- note added: "supply; D5, D6 clamp a rail left open. 100 uF a rail for"
- note added: "the brush hash. ±12 V unloaded, ±8.5 V into a stall; 10 V motor,"
- note added: "the motor's pulses, a green LED per rail, 100 nF at every"
- note added: "this slide pot (T about 33 ms) that is 5 ms, about"
- note added: "through 1k: ±12 V"
- note added: "two probes, A - B, never a ground clip there."
- note added: "±12 V, 0.35 A fuse"
- note removed: "(0.6 A) trips it in 5-10 s, a short in"
- note removed: "(±0.5 V at 0.2 Hz) replaces the knob"
- note removed: "231k with the 22 nF; for the book's rotary motor-pot"
- note removed: "POWER: ±15 V, 1 A (the motor's stall current)."
- note removed: "Quiescent about 10 mA. 100 nF at every op-amp pin."
- note removed: "Series Schottkys against a reversed supply; 100 uF a"
- note removed: "Simulated as drawn (sim/pid_sim.py, the fader modelled from bench measurements): P only rings at 31 Hz when the gain"
- note removed: "about 1 s; the red lamp lights while it"
- note removed: "at a few volts it holds: one transistor takes up to 3.4 W,"
- note removed: "behind it. The 0.35 A PTC opens a full-drive stall (0.6 A)"
- note removed: "in 28 ms with 3 % overshoot. I removes the residual error at low P gain."
- note removed: "in seconds and a short in about one, then resets. A stall"
- note removed: "is tripped. It resets when the drive stops."
- note removed: "nears 100; D equal to P there wants RC = 1 / 2 pi f = 5 ms (RV3 near 231k with 22 nF), and then gain 100 settles"
- note removed: "not in the book. A stall at full drive"
- note removed: "per ampere: two probes, A - B (never a ground clip there)."
- note removed: "rail for the motor's pulses; a green LED per rail."
- note removed: "so they are D2PAKs on 2 oz pours. Across R21 or R22, 1 V"
- note removed: "the brush hash. ±13 V unloaded, ±9 V into a stall; 10 V motor,"
- note removed: "this slide pot (T about 32 ms) that is 5 ms, about"
- note removed: "through 1k: ±13 V"
- note removed: "±13 V, 0.35 A fuse"
- company: Circuit: Hayes & Horowitz, Learning the Art of Electronics (2016), Lab 10L  |  Board: Jason Gallicchio and Claude -> Circuit: Hayes & Horowitz (LAoE, Lab 10L).  Board: J. Gallicchio, Claude
