File: hardware/motorpid.kicad_pcb (KiCad board)
At the start: 2 copper layers, 170 x 120 mm, 106 parts, among them J1 BNC, J2 BNC, J3 BNC, J4 MOTOR + - shield, J5 POT 1 (+) 2 (wiper) 3 (-), J6 +15 / GND / -15, Q1 MJD44H11, Q2 MJD45H11, SW1 TARGET SOURCE, SW2 LOOP, SW3 D IN / OFF, SW4 I IN / OFF, SW5 D CAPACITOR, U1 LM321, U2 LM321, U3 LM321, U4 LM321, U5 LM321, U6 LM321, U7 LM321

Commit message: Fab package, documents, simulation update and chat log for rev A: build passes end to end (ERC 0, 243 circuit checks, DRC 0, fab checks, 23 document claims)
Co-Authored-By: Claude Fable 5.1 <noreply@anthropic.com>
Claude-Session: https://claude.ai/code/session_017Q2PYKR2UewvTfQgKmRJsG
Other:
- board text added: "+ end. If the loop runs away,"
- board text added: "1 (knob), LOOP 1 (open), D OFF 1,"
- board text added: "Both green lamps light."
- board text added: "FADER: motor to MOTOR + GND; track"
- board text added: "GAIN until it rings (~12 Hz),"
- board text added: "I OFF 1, D CAPACITOR 1 (22 nF)."
- board text added: "LAB 10L: the fader's wiper is held"
- board text added: "POSITION must read +7.7 V at the"
- board text added: "POWER: +15, GND, -15 V, 1 A each."
- board text added: "PROBE LOOPS on every node, GND x4."
- board text added: "SQUARE WAVE: TARGET SOURCE 3, feed"
- board text added: "STALL: the 0.35 A fuse opens in"
- board text added: "SWITCHES to start: TARGET SOURCE"
- board text added: "TARGET IN +/-0.5 V at 0.2 Hz."
- board text added: "THEN: LOOP 3 closes it. Raise P"
- board text added: "Trimmers fully anticlockwise."
- board text added: "back to low P, I IN, I GAIN up."
- board text added: "ends to POT + and -, wiper to 2."
- board text added: "seconds, red lamps light; resets."
- board text added: "swap the two motor wires."
- board text added: "switch D IN and turn D GAIN up;"
- board text added: "where TARGET says, by P, D and I."
- board text removed: "(back text to come)"

Commit message: Clockwise arcs over the knob and the three trimmers (Bourns CW = terminal 3; rheostats 1-2, wiper ties under the bodies); handbook's I GAIN direction fixed; Jason's answers recorded: fuse kept, size kept, MSK12C02 travel from its section, fader measurements to make
Co-Authored-By: Claude Fable 5.1 <noreply@anthropic.com>
Claude-Session: https://claude.ai/code/session_017Q2PYKR2UewvTfQgKmRJsG
Parts:
- moved R14 6.38 mm to (111.3, 52.8)
- moved RV3 2.06 mm to (94.5, 79.5)
- moved RV2 1.05 mm to (117.0, 51.5)
- moved C7 1.00 mm to (89.3, 73.5)
Routing:
- net /SUM: track 75.2 -> 68.2 mm
- net /D: track 43.0 -> 48.8 mm
- net Net-(SW4-A): track 71.9 -> 67.7 mm
- net Net-(R14-Pad2): track 6.27 -> 2.25 mm
- net Net-(U3--): track 58.1 -> 56.9 mm
- net GND: track 141.4 -> 140.6 mm
- net Net-(SW3-A): track 70.0 -> 70.5 mm
Other:
- board text added: "D"
- board text added: "GAIN"
- board text added: "↑R ↑D"
- board text added: "↑R ↑P"
- board text added: "↑R ↓I"
- board text added: "↑TARGET"
- board text removed: "D GAIN"

Commit message: Probe loops on BASES, U6 OUT and U7 OUT; LOOP explained on the schematic, front, back and handbook (open = DRIVE from TARGET); ground moved clear of RV4's I; back silkscreen rewritten one item per line with https URL
Co-Authored-By: Claude Opus 5.5 <noreply@anthropic.com>
Claude-Session: https://claude.ai/code/session_017Q2PYKR2UewvTfQgKmRJsG
Parts:
- added TP12: BASES, motorpid:TestPoint_Loop_RH-5019, F.Cu at (162.0, 80.0)
- added TP13: U6 OUT, motorpid:TestPoint_Loop_RH-5019, F.Cu at (141.5, 65.0)
- added TP14: U7 OUT, motorpid:TestPoint_Loop_RH-5019, F.Cu at (29.0, 93.0)
- moved RV4 0.80 mm to (78.7, 100.0)
- moved R17 0.50 mm to (73.0, 97.0)
Routing:
- net Net-(SW4-A): track 67.7 -> 68.5 mm
- net /ERROR: track 90.6 -> 90.1 mm
Other:
- board text added: "1 = 22 nF, for this fader"
- board text added: "1 = off: the 10 uF shorted, so I restarts from zero"
- board text added: "1 = off: the differentiator's output shorted"
- board text added: "1 = open loop"
- board text added: "1 = open: no feedback; DRIVE = P GAIN x TARGET (+ D, I if in)"
- board text added: "1 = the knob"
- board text added: "3 = 100 nF, for the book's slower rotary pot"
- board text added: "3 = D into the sum"
- board text added: "3 = I into the sum"
- board text added: "3 = closed loop"
- board text added: "3 = closed: POSITION fed back, the loop holds TARGET"
- board text added: "3 = the TARGET IN jack"
- board text added: "A stall opens the 0.35 A fuse in seconds; red lamps; it resets itself."
- board text added: "BASES"
- board text added: "Both green lamps light. A reversed supply is blocked: the lamps stay dark."
- board text added: "Check with LOOP open: slide it by hand, POSITION is +7.7 V at the + end."
- board text added: "D IN, raise D GAIN: the ringing dies. Lower P; I IN: the error goes to 0."
- board text added: "FADER: its motor to MOTOR and GND on the MOTOR terminal."
- board text added: "INPUTS"
- board text added: "Its track's two ends to POT + and -, its wiper to the middle pin."
- board text added: "LAB 10L: a PID loop holds a fader (motorized potentiometer) where TARGET says."
- board text added: "LOOP closed and the slider runs to an end and stays: swap the motor leads."
- board text added: "LOOP to 3: the slider follows the knob. Raise P GAIN until it rings."
- board text added: "Never short MOTOR to GND or to a rail. Power off to wire the fader."
- board text added: "OUTPUTS, each through 1k: for a scope, not a load"
- board text added: "P GAIN anticlockwise, D and I off: DRIVE = TARGET"
- board text added: "POSITION OUT: the fader's wiper, buffered. DRIVE OUT: the motor drive."
- board text added: "POWER: +15 V, GND, -15 V on the POWER terminal, 1 A per rail."
- board text added: "START: every switch on 1. P and D GAIN anticlockwise, I GAIN clockwise."
- board text added: "SWITCHES"
- board text added: "TARGET IN jack: a function generator, +/-12 V max."
- board text added: "TARGET SOURCE"
- board text added: "TARGET knob: centre detent = 0 V, clockwise +, up to +/-6.4 V."
- board text added: "TRIMMERS: clockwise = more resistance: more P, more D, but LESS I."
- board text added: "Try a +/-0.5 V square wave at 0.2 Hz: repeatable steps."
- board text added: "U6 OUT"
- board text added: "U7 OUT"
- board text added: "WARNINGS"
- board text added: "https://github.com/gallicchio/motor-pid"
- board text removed: "+ end. If the loop runs away,"
- board text removed: "1 (knob), LOOP 1 (open), D OFF 1,"
- board text removed: "1 = open"
- board text removed: "3 = closed"
- board text removed: "Both green lamps light."
- board text removed: "FADER: motor to MOTOR + GND; track"
- board text removed: "GAIN until it rings (~12 Hz),"
- board text removed: "I OFF 1, D CAPACITOR 1 (22 nF)."
- board text removed: "LAB 10L: the fader's wiper is held"
- board text removed: "POSITION must read +7.7 V at the"
- board text removed: "POWER: +15, GND, -15 V, 1 A each."
- board text removed: "PROBE LOOPS on every node, GND x4."
- board text removed: "SQUARE WAVE: TARGET SOURCE 3, feed"
- board text removed: "STALL: the 0.35 A fuse opens in"
- board text removed: "SWITCHES to start: TARGET SOURCE"
- board text removed: "TARGET IN +/-0.5 V at 0.2 Hz."
- board text removed: "THEN: LOOP 3 closes it. Raise P"
- board text removed: "Trimmers fully anticlockwise."
- board text removed: "back to low P, I IN, I GAIN up."
- board text removed: "ends to POT + and -, wiper to 2."
- board text removed: "github.com/gallicchio/motor-pid"
- board text removed: "seconds, red lamps light; resets."
- board text removed: "swap the two motor wires."
- board text removed: "switch D IN and turn D GAIN up;"
- board text removed: "where TARGET says, by P, D and I."

Commit message: Fader measured and identified: Bourns PSM01-082A-103B2 (taper B2, A+ toward 1), plant refit to Jason's bench numbers (14 ohm, 2-3 V breakaway, 0.16 A running); stick-slip triangle sim; D rule now 234k; 1M trimmers kept; low-drive stall heats the driver (open, warnings added)
Co-Authored-By: Claude Opus 5.5 <noreply@anthropic.com>
Claude-Session: https://claude.ai/code/session_017Q2PYKR2UewvTfQgKmRJsG
Other:
- board text added: "A stall at a few volts does not: it heats the driver. Seconds, not minutes."
- board text added: "A stall at full drive opens the 0.35 A fuse in seconds (red lamps); it resets."
- board text added: "FADER (Bourns PSM01-082A-103B2): motor A to MOTOR, motor B to GND."
- board text added: "Track 1, 2, 3 to POT 1 (+), 2 (wiper), 3 (-): the numbers match."
- board text added: "Try +/-3 V: a 0.2 Hz square wave for steps, a 0.05 Hz triangle for stick-slip."
- board text removed: "A stall opens the 0.35 A fuse in seconds; red lamps; it resets itself."
- board text removed: "FADER: its motor to MOTOR and GND on the MOTOR terminal."
- board text removed: "Its track's two ends to POT + and -, its wiper to the middle pin."
- board text removed: "Try a +/-0.5 V square wave at 0.2 Hz: repeatable steps."
Changed lines of the file:
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@@
 		)
 	)
-	(gr_text "Try a +/-0.5 V square wave at 0.2 Hz: repeatable steps."
+	(gr_text "Try +/-3 V: a 0.2 Hz square wave for steps, a 0.05 Hz triangle for stick-slip."
 		(at 64 70.2 0)
 		(layer "B.SilkS")
@@
 		)
 	)
-	(gr_text "Its track's two ends to POT + and -, its wiper to the middle pin."
+	(gr_text "Track 1, 2, 3 to POT 1 (+), 2 (wiper), 3 (-): the numbers match."
 		(at 67 60.6 0)
 		(layer "B.SilkS")
@@
 		)
 	)
-	(gr_text "A stall opens the 0.35 A fuse in seconds; red lamps; it resets itself."
+	(gr_text "A stall at full drive opens the 0.35 A fuse in seconds (red lamps); it resets."
 		(at 67 102.2 0)
 		(layer "B.SilkS")
@@
 		)
 	)
+	(gr_text "A stall at a few volts does not: it heats the driver.  Seconds, not minutes."
+		(at 67 103.8 0)
+		(layer "B.SilkS")
+		(effects
+			(font
+				(size 0.9 0.9)
+				(thickness 0.15)
+			)
+			(justify left mirror)
+		)
+	)
 	(gr_text "Never short MOTOR to GND or to a rail.  Power off to wire the fader."
-		(at 67 103.8 0)
+		(at 67 105.4 0)
 		(layer "B.SilkS")
 		(effects
@@
 		)
 	)
-	(gr_text "FADER: its motor to MOTOR and GND on the MOTOR terminal."
+	(gr_text "FADER (Bourns PSM01-082A-103B2): motor A to MOTOR, motor B to GND."
 		(at 70 59 0)
 		(layer "B.SilkS")

Commit message: Push-pull on D2PAKs and 2 oz copper (Jason's choice): MJB44H11/MJB45H11 in pours that are their heatsink, 120/122 C junctions in the worst stall, checked on the board as built
- parts: MJB44H11T4G C233689 / MJB45H11T4G C154570, TO-263-2; JLCPCB draws
  them turned 180 (CPL +180, datum 2.45 mm toward the leads, predicted)
- layout: Q1/Q2 symbols drawn round the leads with the tab capping the
  circle; pours fill the MOTOR DRIVER box round each tab (836 / 670 mm2);
  R21/R22 in two columns; D3/D4 with their rail ends in the pours; snubber
  under DRIVE; BASES crosses Q2's emitter wire on the back (one hop: the
  mirrored PNP makes the crossing topological)
- back runs moved off the plane under the pours: lower stages' +15 V from
  the rail, Q2's -15 V up the board edge, U6 V- and the track's -15 V from
  Q2's pour
- 2 oz: clearance and min track 0.21 mm, board stackup 0.07 mm copper,
  order form says 2 oz, bare-board cost x1.5
- sim/thermal.py --board: the model on the filled pours and the plane with
  its cuts; make.py fails above 125 C at the junction; sim/thermal.json
- pid_sim refuses a transistor it has no model for (a stale netlist
  silently simulated the wrong part once)
- docs: decision recorded, 5 new build-checked claims, HOT on both pours,
  warnings softened from "seconds" to "the copper is hot"

ERC 0, 249 checks, DRC 0, fab checks, 30/30 claims, BUILD OK.

Co-Authored-By: Claude Opus 5.5 <noreply@anthropic.com>
Claude-Session: https://claude.ai/code/session_017Q2PYKR2UewvTfQgKmRJsG
Parts:
- Q1: value MJD44H11 -> MJB44H11; footprint Package_TO_SOT_SMD:TO-252-2 -> Package_TO_SOT_SMD:TO-263-2
- Q2: value MJD45H11 -> MJB45H11; footprint Package_TO_SOT_SMD:TO-252-2 -> Package_TO_SOT_SMD:TO-263-2
- moved TP12 32.2 mm to (146.0, 52.0)
- moved D4 9.74 mm to (164.8, 62.6), turned to -90 degrees
- moved D3 8.87 mm to (164.8, 55.4)
- moved C10 8.50 mm to (156.5, 62.0), turned to 180 degrees
- moved Q2 7.76 mm to (154.0, 80.0)
- moved R21 4.98 mm to (156.5, 56.0)
- moved Q1 4.83 mm to (154.0, 39.1)
- moved R20 4.03 mm to (160.0, 62.0), turned to 180 degrees
- moved R22 0.54 mm to (151.5, 62.0)
Routing:
- net -15V: track 747.8 -> 614.9 mm, vias 20 -> 21
- net +15V: track 591.0 -> 511.1 mm
- net /BASES: track 106.2 -> 54.1 mm, vias 0 -> 2
- net Net-(Q2-E): track 4.78 -> 7.42 mm
- net /DRIVE: track 133.1 -> 130.8 mm
- net Net-(Q1-E): track 4.78 -> 6.33 mm
- net Net-(C10-Pad1): track 2.64 -> 1.64 mm
- net GND: track 140.3 -> 139.7 mm
Other:
- board text added: "A stall at a few volts does not: the copper marked HOT reaches about 90 C."
- board text added: "C10 100nF"
- board text added: "HOT if the"
- board text added: "MJB44H11"
- board text added: "MJB45H11"
- board text added: "R20 10R"
- board text added: "motor stalls"
- board text removed: "A stall at a few volts does not: it heats the driver. Seconds, not minutes."
- board text removed: "MJD44H11"
- board text removed: "MJD45H11"

Commit message: Review round 1 applied (Jason): the patch, the fuse between the push-pull and DRIVE, the integrator's capacitor a 1 uF polypropylene film
- patch_round1.diff as it stood: switch-end numbers, three vias each end of Q2's -15 V run,
  TARGET IN at +/-3 V, standoffs, handbook table and gains recipe, R4's run off the URL,
  sheet notes; its "DRIVE ahead of the fuse" warnings rewritten for the moved fuse
- F1 right after R21/R22: the feedback, the DRIVE loop, DRIVE OUT and the motor terminal
  behind it; clamps and snubber stay at the transistors; MOTOR merged into DRIVE (17 loops);
  check_circuit asserts what is ahead of the fuse and that no loop or connector is
- C8: Panasonic ECWF2W105JA 1 uF PP film (C242107), generated footprint and model; RC 1 ms
  to 1 s across the 1M trimmer; the LM321's bias current through 1M (45 mV) in a check
- sim: motor on DRIVE, Q1's power from its own pins (3.4 W; the old 3.7 included R21),
  I runs at 1M and 50k; thermal check keeps 3.7 W as a bound, 120/122 C
- fab notes: D4's cathode and C12's stripe were drawn the wrong way; the 1R's BOM note
- the review brief describes the patched board; reviews README and the report's addendum
- ERC 0, 252 checks, DRC 0, fab checks, 30/30 claims

Co-Authored-By: Claude Opus 5.5 <noreply@anthropic.com>
Claude-Session: https://claude.ai/code/session_017Q2PYKR2UewvTfQgKmRJsG
Parts:
- removed TP14: U7 OUT, motorpid:TestPoint_Loop_RH-5019
- C8: value 10uF -> 1uF; footprint Capacitor_SMD:C_0805_2012Metric -> motorpid:C_Film_Panasonic_ECWF_L18.1mm_W9.3mm_P15.00mm
- TP11: value MOTOR -> BASES
- TP12: value BASES -> U6 OUT
- TP13: value U6 OUT -> U7 OUT
- moved TP13 115.9 mm to (29.0, 93.0)
- moved TP11 47.3 mm to (146.0, 52.0), turned to 90 degrees
- moved TP12 13.8 mm to (141.5, 65.0)
- moved C8 4.66 mm to (93.7, 110.3)
Connections:
- D3 pad 2: /DRIVE -> Net-(D3-A)
- D4 pad 1: /DRIVE -> Net-(D3-A)
- F1 pad 1: /DRIVE -> Net-(D3-A)
- F1 pad 2: /MOTOR -> /DRIVE
- J4 pad 1: /MOTOR -> /DRIVE
- LED3 pad 2: /MOTOR -> /DRIVE
- LED4 pad 1: /MOTOR -> /DRIVE
- R20 pad 1: /DRIVE -> Net-(D3-A)
- R21 pad 2: /DRIVE -> Net-(D3-A)
- R22 pad 1: /DRIVE -> Net-(D3-A)
- R23 pad 1: /DRIVE -> Net-(D3-A)
- TP11 pad 1: /MOTOR -> /BASES
- TP12 pad 1: /BASES -> Net-(C9-Pad2)
- TP13 pad 1: Net-(C9-Pad2) -> Net-(U7--)
Routing:
- net Net-(D3-A): track 0.00 -> 63.7 mm
- net /MOTOR: track 44.5 -> 0.00 mm
- net /DRIVE: track 130.8 -> 98.6 mm
- net Net-(J3-In): track 70.3 -> 81.9 mm
- net -15V: track 614.9 -> 624.5 mm, vias 21 -> 25
- net Net-(SW4-A): track 68.5 -> 78.1 mm
- net /I: track 31.6 -> 26.2 mm
Other:
- board text added: "1"
- board text added: "1 = off: the 1 uF shorted, so I restarts from zero"
- board text added: "3"
- board text added: "A stall at a few volts does not: HOT copper reaches 90 C, so use the standoffs."
- board text added: "A stall at full drive or a short to GND opens the fuse (red lamps); it resets."
- board text added: "Never short MOTOR or DRIVE to a rail. Power off to wire the fader."
- board text added: "film"
- board text added: "±3 V at 0.2 Hz replaces the knob"
- board text removed: "1 = off: the 10 uF shorted, so I restarts from zero"
- board text removed: "A stall at a few volts does not: the copper marked HOT reaches about 90 C."
- board text removed: "A stall at full drive opens the 0.35 A fuse in seconds (red lamps); it resets."
- board text removed: "Never short MOTOR to GND or to a rail. Power off to wire the fader."
- board text removed: "±0.5 V at 0.2 Hz replaces the knob"
